Commit message: check the urdf limits

File: schunk_description/urdf/lwa4p_extended/lwa4p_extended.urdf.xacro (robot description, xacro)
@@ -103,5 +103,5 @@
       <axis xyz="0 0 1"/>
       <dynamics damping="0" friction="0"/>
-      <limit effort="48" velocity="1.57" lower="${-1.91 + safety_offset}" upper="${1.91 - safety_offset}"/>   <!--Theoretical limit +/-170 , Real Limit +/- 110 (self collision)-->
+      <limit effort="48" velocity="1.57" lower="${-1.8 + safety_offset}" upper="${1.8 - safety_offset}"/>   <!--Theoretical limit +/-170 , Real Limit +/- 110 (self collision)-->
       <!--safety_controller k_position="20" k_velocity="50" soft_lower_limit="${-2.0943 + 0.01}" soft_upper_limit="${2.0943 - 0.01}" /-->
     </joint>
@@ -199,5 +199,5 @@
       <axis xyz="0 0 1" />
       <dynamics damping="0" friction="0"/>
-      <limit effort="48" velocity="1.57" lower="${-2.96 + safety_offset}" upper="${2.96 - safety_offset}"/>   <!--Theoretical limit +/-170 , Real Limit +/- 170-->
+      <limit effort="48" velocity="1.57" lower="${-2.76 + safety_offset}" upper="${2.76 - safety_offset}"/>   <!--Theoretical limit +/-170 , Real Limit +/- 170-->
       <!--safety_controller k_position="20" k_velocity="25" soft_lower_limit="${-M_PI + 0.01}" soft_upper_limit="${M_PI - 0.01}" /-->
     </joint>
@@ -231,5 +231,5 @@
       <axis xyz="0 0 1" />
       <dynamics damping="0" friction="0"/>
-      <limit effort="15" velocity="2.09" lower="${-2.96 + safety_offset}" upper="${2.96 - safety_offset}"/>   <!--Theoretical limit +/-170 , Real Limit -140/+170 (self collision)-->
+      <limit effort="15" velocity="2.09" lower="${-2.4 + safety_offset}" upper="${2.4 - safety_offset}"/>   <!--Theoretical limit +/-170 , Real Limit -140/+170 (self collision)-->
       <!--safety_controller k_position="20" k_velocity="25" soft_lower_limit="${-2.0943951 + 0.01}" soft_upper_limit="${2.0943951 - 0.01}" /-->
     </joint>
